File: modules/VCS/mount/mount.kicad_pcb (KiCad board)
At the start: 2 copper layers, 60.6 x 111.8 mm, 34 parts, among them J1 FALL CV, J10 OUT, J11 BIPOLAR OUT, J2 BOTH CV, J3 RISE CV, J4 CV (1V/OCT), J5 IN, J6 TRIGGER, J7 Conn_01x21_Male, J8 END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

Commit message: update schema
Parts:
- added D6: 1N4148, Diode_THT:D_DO-35_SOD27_P7.62mm_Horizontal, F.Cu at (53.2, 35.3)
- added J12: Conn_01x08_Female, Connector_PinHeader_2.54mm:PinHeader_1x08_P2.54mm_Vertical, F.Cu at (28.3, 72.1)
- added Q3: 2N3904, Package_TO_SOT_THT:TO-92_Inline, F.Cu at (66.9, 28.7)
- added R39: 150k, Resistor_THT:R_Axial_DIN0207_L6.3mm_D2.5mm_P10.16mm_Horizontal, F.Cu at (53.2, 27.5)
- added R44: 1k, Resistor_THT:R_Axial_DIN0207_L6.3mm_D2.5mm_P10.16mm_Horizontal, F.Cu at (53.2, 31.5)
Connections:
- D1 pad 1: /LED -> Net-(D1-Pad1)
- J1 pad TN: Net-(J1-PadTN) -> (no net)
- J10 pad TN: Net-(J10-PadTN) -> (no net)
- J11 pad TN: Net-(J11-PadTN) -> (no net)
- J2 pad TN: Net-(J2-PadTN) -> (no net)
- J3 pad TN: Net-(J3-PadTN) -> (no net)
- J4 pad TN: Net-(J4-PadTN) -> (no net)
- J5 pad TN: Net-(J5-PadTN) -> (no net)
- J6 pad TN: Net-(J6-PadTN) -> (no net)
- J7 pad 1: /RISE -> GND
- J7 pad 10: /CV -> (no net)
- J7 pad 11: /BIPOLAR_OUT -> (no net)
- J7 pad 12: /NET_1 -> (no net)
- J7 pad 13: /LED -> /CV
- J7 pad 14: /OUT -> /BIPOLAR_OUT
- J7 pad 15: /AC_OUT -> /NET_1
- J7 pad 16: /CYCLE_2 -> (no net)
- J7 pad 17: /CYCLE_1 -> /OUT
- J7 pad 18: /TRIGGER -> /AC_OUT
- J7 pad 19: +15V -> /CYCLE_2
- J7 pad 2: /FALL_1 -> +15V
- J7 pad 20: -15V -> /CYCLE_1
- J7 pad 21: GND -> /TRIGGER
- J7 pad 3: /FALL -> -15V
- J7 pad 4: /RISE_2 -> (no net)
- J7 pad 5: /FALL_2 -> (no net)
- J7 pad 6: /IN -> (no net)
- J7 pad 7: /FALL_RATE -> (no net)
- J7 pad 8: /RISE_1 -> (no net)
- J7 pad 9: /RISE_RATE -> /IN
- J8 pad TN: Net-(J8-PadTN) -> (no net)
- J9 pad TN: Net-(J9-PadTN) -> (no net)
- SW1 pad 3: Net-(SW1-Pad3) -> (no net)
- SW2 pad 3: Net-(SW2-Pad3) -> (no net)
- SW3 pad 3: Net-(SW3-Pad3) -> (no net)
Routing:
- net GND: track 229.6 -> 85.6 mm
- net +15V: track 110.4 -> 0.00 mm
- net /CV: track 95.3 -> 0.00 mm, vias 1 -> 0
- net /FALL_2: track 94.1 -> 0.00 mm
- net /NET_1: track 79.9 -> 0.00 mm
- net /RISE: track 100.4 -> 23.1 mm
- net /TRIGGER: track 63.5 -> 0.00 mm
- net /LED: track 60.4 -> 0.00 mm
- net /FALL: track 64.7 -> 5.08 mm
- net /RISE_1: track 58.7 -> 8.87 mm, vias 1 -> 0
- net /RISE_2: track 61.4 -> 11.7 mm
- net /FALL_RATE: track 74.2 -> 40.5 mm, vias 1 -> 0
- net /FALL_1: track 79.5 -> 57.5 mm
- net /RISE_RATE: track 36.8 -> 30.9 mm
