File: modules/ssg/main/main.kicad_pcb (KiCad board)
At the start: 2 copper layers, 60.6 x 111.8 mm, 104 parts, among them J1 IDC Header, J2 Conn_01x12_Female, J3 Conn_01x09_Female, Q1 PN4250, Q2 PN4250, Q3 J201, Q4 J201, U1 TL072, U2 LM3900, U3 LM3900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

Commit message: R02
Parts:
- R28: value 1m -> 1M
Connections:
- U5 pad 1: Net-(U5-Pad1) -> (no net)
- U5 pad 8: Net-(U5-Pad8) -> (no net)
- U6 pad 1: Net-(U6-Pad1) -> (no net)
- U6 pad 8: Net-(U6-Pad8) -> (no net)
- U7 pad 1: Net-(U7-Pad1) -> (no net)
- U7 pad 5: Net-(U7-Pad5) -> (no net)
- U7 pad 8: Net-(U7-Pad8) -> (no net)
