File: modules/bpf/panel/panel.kicad_pcb (KiCad board)
At the start: 2 copper layers, 80.9 x 133.4 mm, 23 parts

Commit message: update schematica
Parts:
- removed H11: IN_2_b, elektrophon:panel_jack
- removed H2: IN_1_b, elektrophon:panel_jack
- H1: value IN_1_a -> IN_1
- H10: value IN_2_a -> IN_2
- H15: value IN_3_a -> IN_3
- H16: value IN_3_b -> IN
- moved H20 86.2 mm to (35.6, 111.8)
- moved H21 57.5 mm to (55.9, 111.8)
- moved H16 45.4 mm to (35.6, 50.8)
- moved H22 28.7 mm to (76.2, 111.8)
- moved H13 20.3 mm to (55.9, 91.4)
- moved H18 20.3 mm to (76.2, 91.4)
- moved H4 20.3 mm to (35.6, 91.4)
- moved H12 20.3 mm to (55.9, 71.1)
- moved H17 20.3 mm to (76.2, 71.1)
- moved H23 20.3 mm to (76.2, 132.1)
- moved H3 20.3 mm to (35.6, 71.1)
- moved H19 13.5 mm to (62.7, 132.1)
- moved H1 13.5 mm to (49.1, 50.8)
- moved H14 6.77 mm to (49.1, 132.1)
- moved H10 6.77 mm to (62.7, 50.8)
