File: modules/resonanz/mount/mount.kicad_pcb (KiCad board)
At the start: 2 copper layers, 80.9 x 111.8 mm, 43 parts, among them J1 AudioJack2_SwitchT, J10 AudioJack2_SwitchT, J11 Conn_01x26_Male, J12 Conn_01x05_Male, J2 AudioJack2_SwitchT, J3 AudioJack2_SwitchT, J4 AudioJack2_SwitchT, J5 AudioJack2_SwitchT, J6 AudioJack2_SwitchT, J7 AudioJack2_SwitchT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

Commit message: update schema
Parts:
- removed the REF** at (57.4, 149.9)
Connections:
- RV2 pad 1: FREQ_1_a -> FREQ_1_b
- RV2 pad 3: FREQ_1_b -> FREQ_1_a
- RV2 pad 4: FREQ_1_c -> OUT_1
- RV2 pad 6: OUT_1 -> FREQ_1_c
- RV4 pad 1: FREQ_2_a -> FREQ_2_b
- RV4 pad 3: FREQ_2_b -> FREQ_2_a
- RV4 pad 4: FREQ_2_c -> OUT_2
- RV4 pad 6: OUT_2 -> FREQ_2_c
- RV6 pad 1: FREQ_3_a -> FREQ_3_b
- RV6 pad 3: FREQ_3_b -> FREQ_3_a
- RV6 pad 4: FREQ_3_c -> OUT_3
- RV6 pad 6: OUT_3 -> FREQ_3_c
- RV8 pad 1: FREQ_4_a -> FREQ_4_b
- RV8 pad 3: FREQ_4_b -> FREQ_4_a
- RV8 pad 4: FREQ_4_c -> OUT_4
- RV8 pad 6: OUT_4 -> FREQ_4_c
Routing:
- net FREQ_3_a: track 27.7 -> 37.8 mm
- net FREQ_2_c: track 27.8 -> 37.0 mm
- net FREQ_3_c: track 26.7 -> 34.9 mm
- net FREQ_4_c: track 28.8 -> 35.6 mm
- net FREQ_4_b: track 35.8 -> 29.4 mm
- net FREQ_2_a: track 26.8 -> 33.2 mm
- net RES_3: track 57.4 -> 51.5 mm
- net FREQ_4_a: track 33.5 -> 39.3 mm
- net RES_1: track 58.4 -> 52.7 mm
- net FREQ_1_a: track 29.8 -> 35.4 mm
- net FREQ_1_c: track 30.0 -> 35.0 mm
- net FREQ_2_b: track 36.0 -> 32.4 mm
- net FREQ_1_b: track 38.1 -> 34.5 mm
- net FREQ_3_b: track 33.8 -> 30.3 mm
- net OUT_4: track 93.7 -> 91.6 mm
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
Commit message: update resonanz
Parts:
- added REF**: elektrophon logo, elektrophon:elektrophon logo, F.Cu at (55.6, 149.7)
- R1, R11, R5, R7: value 4k7 -> 470
