File: content/adsr/panel/panel.kicad_pcb (KiCad board)
At the start: 2 copper layers, 40.3 x 133.4 mm, 7 parts

Commit message: add kraft
Changed lines of the file:
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@@
-(kicad_pcb (version 20171130) (host pcbnew 5.1.6-c6e7f7d~86~ubuntu20.04.1)
+(kicad_pcb (version 20171130) (host pcbnew 5.1.10)
   (general
     (thickness 1.6)
@@
       (effects (font (size 1 1) (thickness 0.15)))
     )
+    (fp_circle (center 0 0) (end 4.2 0) (layer F.CrtYd) (width 0.05))
     (fp_circle (center 0 0) (end 4 0) (layer Cmts.User) (width 0.15))
-    (fp_circle (center 0 0) (end 4.2 0) (layer F.CrtYd) (width 0.05))
-    (pad "" np_thru_hole circle (at 0 0) (size 6.4 6.4) (drill 6.4) (layers *.Cu *.Mask))
+    (pad "" thru_hole circle (at 0 0) (size 6.4 6.4) (drill 6.4) (layers *.Cu *.Mask))
     (model "${KIPRJMOD}/../../../lib/kicad/models/PJ301M-12 Thonkiconn v0.2.stp"
       (offset (xyz 0 0.8 -10.5))
@@
       (effects (font (size 1 1) (thickness 0.15)))
     )
-    (fp_circle (center 0 0) (end 6.35 0) (layer Cmts.User) (width 0.15))
-    (fp_circle (center 0 0) (end 6.6 0) (layer F.CrtYd) (width 0.05))
-    (pad "" np_thru_hole circle (at 0 0) (size 7.4 7.4) (drill 7.4) (layers *.Cu *.Mask))
+    (fp_circle (center 0 0) (end 6.6 0) (layer F.CrtYd) (width 0.05))
+    (fp_circle (center 0 0) (end 6.35 0) (layer Cmts.User) (width 0.15))
+    (pad "" thru_hole circle (at 0 0) (size 7.4 7.4) (drill 7.4) (layers *.Cu *.Mask))
     (model ${KIPRJMOD}/../../../lib/kicad/models/ALPHA-RD901F-40.step
       (offset (xyz 0 0.5 -12))
@@
       (effects (font (size 1 1) (thickness 0.15)))
     )
-    (fp_circle (center 0 0) (end 6.35 0) (layer Cmts.User) (width 0.15))
-    (fp_circle (center 0 0) (end 6.6 0) (layer F.CrtYd) (width 0.05))
-    (pad "" np_thru_hole circle (at 0 0) (size 7.4 7.4) (drill 7.4) (layers *.Cu *.Mask))
+    (fp_circle (center 0 0) (end 6.6 0) (layer F.CrtYd) (width 0.05))
+    (fp_circle (center 0 0) (end 6.35 0) (layer Cmts.User) (width 0.15))
+    (pad "" thru_hole circle (at 0 0) (size 7.4 7.4) (drill 7.4) (layers *.Cu *.Mask))
     (model ${KIPRJMOD}/../../../lib/kicad/models/ALPHA-RD901F-40.step
       (offset (xyz 0 0.5 -12))
@@
       (effects (font (size 1 1) (thickness 0.15)))
     )
-    (fp_circle (center 0 0) (end 6.35 0) (layer Cmts.User) (width 0.15))
-    (fp_circle (center 0 0) (end 6.6 0) (layer F.CrtYd) (width 0.05))
-    (pad "" np_thru_hole circle (at 0 0) (size 7.4 7.4) (drill 7.4) (layers *.Cu *.Mask))
+    (fp_circle (center 0 0) (end 6.6 0) (layer F.CrtYd) (width 0.05))
+    (fp_circle (center 0 0) (end 6.35 0) (layer Cmts.User) (width 0.15))
+    (pad "" thru_hole circle (at 0 0) (size 7.4 7.4) (drill 7.4) (layers *.Cu *.Mask))
     (model ${KIPRJMOD}/../../../lib/kicad/models/ALPHA-RD901F-40.step
       (offset (xyz 0 0.5 -12))
@@
       (effects (font (size 1 1) (thickness 0.15)))
     )
-    (fp_circle (center 0 0) (end 6.35 0) (layer Cmts.User) (width 0.15))
-    (fp_circle (center 0 0) (end 6.6 0) (layer F.CrtYd) (width 0.05))
-    (pad "" np_thru_hole circle (at 0 0) (size 7.4 7.4) (drill 7.4) (layers *.Cu *.Mask))
+    (fp_circle (center 0 0) (end 6.6 0) (layer F.CrtYd) (width 0.05))
+    (fp_circle (center 0 0) (end 6.35 0) (layer Cmts.User) (width 0.15))
+    (pad "" thru_hole circle (at 0 0) (size 7.4 7.4) (drill 7.4) (layers *.Cu *.Mask))
     (model ${KIPRJMOD}/../../../lib/kicad/models/ALPHA-RD901F-40.step
       (offset (xyz 0 0.5 -12))
@@
       (effects (font (size 1 1) (thickness 0.15)))
     )
+    (fp_circle (center 0 0) (end 4.2 0) (layer F.CrtYd) (width 0.05))
     (fp_circle (center 0 0) (end 4 0) (layer Cmts.User) (width 0.15))
-    (fp_circle (center 0 0) (end 4.2 0) (layer F.CrtYd) (width 0.05))
-    (pad "" np_thru_hole circle (at 0 0) (size 6.4 6.4) (drill 6.4) (layers *.Cu *.Mask))
+    (pad "" thru_hole circle (at 0 0) (size 6.4 6.4) (drill 6.4) (layers *.Cu *.Mask))
     (model "${KIPRJMOD}/../../../lib/kicad/models/PJ301M-12 Thonkiconn v0.2.stp"
       (offset (xyz 0 0.8 -10.5))
