File: content/produkt/mount/mount.kicad_pcb (KiCad board)
At the start: 2 copper layers, 40.3 x 108.2 mm, 47 parts, among them J1 IN_X, J2 IN_Y, J3 OUT, J4 Conn_01x08_Male, J5 IN_X, J6 IN_Y, J7 OUT, Q1 MMBT3904, Q2 MMBT3904, Q3 MMBT3904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

Commit message: update pcb
Parts:
- added J8: Conn_01x03_Male, Connector_PinSocket_2.54mm:PinSocket_1x03_P2.54mm_Vertical, B.Cu at (88.9, 114.3)
- added REF**: elektrophon logo, elektrophon:elektrophon logo, F.Cu at (53.6, 70.4)
- D10, Q2, Q3, Q6, R4, R5, R6: moved to B.Cu
- J4: value Conn_01x08_Male -> Conn_01x05_Male; footprint Connector_PinHeader_2.54mm:PinHeader_1x08_P2.54mm_Vertical -> Connector_PinSocket_2.54mm:PinSocket_1x05_P2.54mm_Vertical; moved to B.Cu
- moved R14 92.2 mm to (67.5, 157.0)
- moved J1 83.8 mm to (61.0, 66.0)
- moved J7 83.8 mm to (81.3, 147.3)
- moved Q5 80.1 mm to (87.4, 147.3), turned to 270 degrees
- moved R12 78.2 mm to (68.6, 148.8)
- moved R11 74.2 mm to (87.4, 143.3)
- moved R3 71.8 mm to (67.1, 71.1), turned to 180 degrees
- moved R13 68.1 mm to (87.4, 140.2)
- moved R7 48.2 mm to (67.5, 111.8), turned to 180 degrees
- moved D10 47.9 mm to (68.1, 144.8)
- moved D6 46.4 mm to (86.9, 99.1), turned to 180 degrees
- moved J2 45.4 mm to (61.0, 106.7)
- moved RV1 45.4 mm to (61.0, 86.4)
- moved RV4 45.4 mm to (81.3, 127.0)
- moved R8 45.2 mm to (87.4, 102.1), turned to 180 degrees
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Routing:
- net +5V: track 0.00 -> 180.1 mm, vias 0 -> 5
- net Net-(J3-PadT): track 0.00 -> 125.1 mm
- net OUTa: track 0.00 -> 66.9 mm
- net OUTb: track 0.00 -> 46.7 mm
- net Ya: track 0.00 -> 43.2 mm
- net /IN2y: track 0.00 -> 35.6 mm
- net /IN2x: track 0.00 -> 31.0 mm
- net /IN1y: track 0.00 -> 29.6 mm
- net /IN1x: track 0.00 -> 29.1 mm
- net Xb: track 0.00 -> 26.5 mm
- net Yb: track 0.00 -> 20.8 mm
- net Net-(D2-Pad1): track 0.00 -> 16.6 mm
- net Net-(D8-Pad2): track 0.00 -> 14.6 mm
- net Net-(D7-Pad2): track 0.00 -> 12.4 mm
- net Net-(D3-Pad2): track 0.00 -> 12.0 mm
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- added copper zone on B.Cu, net GND

Commit message: update PCB's
Parts:
- D11, D12: value LED -> LED (Red)
- D3, D4, D7, D8: value LED -> LED (Green)
- R1, R2: footprint Resistor_THT:R_Axial_DIN0207_L6.3mm_D2.5mm_P10.16mm_Horizontal -> Resistor_THT:R_Axial_DIN0204_L3.6mm_D1.6mm_P5.08mm_Horizontal
- moved R2 5.59 mm to (73.2, 146.8)
- moved R1 5.59 mm to (53.8, 146.3)
Routing:
- net OUTa: track 66.9 -> 74.6 mm, vias 0 -> 1
- net OUTb: track 46.7 -> 52.3 mm
