File: content/kontur/mount/mount.kicad_pcb (KiCad board)
At the start: 2 copper layers, 40.3 x 108.2 mm, 53 parts, among them J1 Conn_01x09_Male, J2 Conn_01x07_Male, J3 AudioJack2_SwitchT, J4 AudioJack2_SwitchT, J5 AudioJack2_SwitchT, J6 AudioJack2_SwitchT, J7 AudioJack2_SwitchT, J8 AudioJack2_SwitchT, Q1 MMBT3904, Q2 MMBT3904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

Commit message: finalize PCB
Parts:
- added H1: MountingHole, MountingHole:MountingHole_2.2mm_M2, F.Cu at (53.3, 53.3)
- added REF**: elektrophon logo, elektrophon:elektrophon logo, F.Cu at (89.2, 118.6)
- D11, D12, D7, D8: value LED -> LED (Red)
- D3, D4: value LED -> LED (Yellow)
- J1: value Conn_01x09_Male -> 01x09 Male
- J2: value Conn_01x07_Male -> 01x07 Male
