File: content/oberwelle/main/main.kicad_pcb (KiCad board)
At the start: 2 copper layers, 60.6 x 111.8 mm, 135 parts, among them J1 IDC Header, J2 Conn_01x07_Female, J3 Conn_01x06_Female, Q1 BC557, U1 TL072, U2 TL072, U3 CA3080, U4 TL072, U5 TL072, U6 LM3900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

Commit message: update schemas
Parts:
- moved R56 4.96 mm to (43.1, 110.1), turned to 180 degrees
Connections:
- R42 pad 1: GND -> -15V
- R49 pad 1: GND -> -15V
- R56 pad 1: GND -> -15V
Routing:
- net -15V: track 376.5 -> 399.0 mm
- net +15V: track 319.5 -> 331.4 mm
- net GND: track 698.2 -> 691.7 mm
- net Net-(R52-Pad2): track 35.1 -> 37.3 mm
