File: src/hall/panel/panel.kicad_sch (KiCad schematic)
At the start: 12 parts

Commit message: cleanup files
Parts:
- removed H5: IN3, elektrophon:panel_jack, symbol Mechanical:MountingHole
- H1: value (none) -> IN1; footprint elektrophon:MountingHole_Panel_3.2mm_M3 -> elektrophon:panel_jack
- H10: value ATTEN_2 -> compress; footprint elektrophon:panel_potentiometer -> elektrophon:panel_led_monitor
- H11: value ATTEN_3 -> (none); footprint elektrophon:panel_potentiometer -> elektrophon:MountingHole_Panel_3.2mm_M3
- H12: value ATTEN_4 -> (none); footprint elektrophon:panel_potentiometer -> elektrophon:MountingHole_Panel_3.2mm_M3
- H2: value (none) -> IN2; footprint elektrophon:MountingHole_Panel_3.2mm_M3 -> elektrophon:panel_jack
- H3: value IN1 -> FDBK
- H4: value IN2 -> OUT
- H6: value IN4 -> level; footprint elektrophon:panel_jack -> elektrophon:panel_potentiometer
- H7: value OUT_a -> bass; footprint elektrophon:panel_jack -> elektrophon:panel_potentiometer
- H8: value OUT_b -> treble; footprint elektrophon:panel_jack -> elektrophon:panel_potentiometer
- H9: value ATTEN_1 -> mix
Other:
- title: cp3 -> pentode vca
- moved on the sheet: H1, H10, H11, H12, H2, H3, H4, H6, H7, H8, H9

Commit message: update to Kicad8
Parts:
- H1, H10, H11, H12, H2, H3, H4, H6, H7, H8, H9: now left out of the parts list
